File: PCB/Keyboard/Altair.kicad_sch (KiCad schematic)
At the start: 6 parts, among them J1 Conn_01x02_Socket, SW97 SW_Nidec_CAS-120A1, SW98 RotaryEncoder_Switch, SW99 SW_Push, U1 SuperMini nRF52840

Commit message: inprocessing
Connections:
- net at U1.11 (P1.04-LF): now also SW97.2 (B)
- net at U1.12 (P1.06-LF): no longer SW97.2 (B)
Changed lines of the file:
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@@
+	(wire
+		(pts
+			(xy 44.45 97.79) (xy 50.8 97.79)
+		)
+		(stroke
+			(width 0)
+			(type default)
+		)
+	)
+	(wire
+		(pts
+			(xy 50.8 97.79) (xy 50.8 109.22)
+		)
+		(stroke
+			(width 0)
+			(type default)
+		)
+	)
+	(wire
+		(pts
+			(xy 44.45 93.98) (xy 69.85 93.98)
+		)
+		(stroke
+			(width 0)
+			(type default)
+		)
+	)
 	(wire
 		(pts
@@
 	(wire
 		(pts
-			(xy 50.8 109.22) (xy 50.8 96.52)
+			(xy 44.45 97.79) (xy 44.45 93.98)
 		)
 		(stroke
@@
 		)
 		(stroke
-			(width 0)
-			(type default)
-		)
-	)
-	(wire
-		(pts
-			(xy 50.8 96.52) (xy 69.85 96.52)
-		)
-		(stroke

Commit message: add sample
Connections:
- net at U1.14 (GND): no longer SW99.1
- net at U1.15 (RST): no longer SW99.2
- new net GND: SW99.2
- new net RST: SW99.1
Other:
- moved on the sheet: SW99
Changed lines of the file:
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@@
 	(wire
 		(pts
-			(xy 107.95 71.12) (xy 115.57 71.12)
+			(xy 147.32 78.74) (xy 143.51 78.74)
 		)
 		(stroke
@@
 	(wire
 		(pts
-			(xy 147.32 78.74) (xy 143.51 78.74)
+			(xy 44.45 97.79) (xy 44.45 93.98)
 		)
 		(stroke
@@
 	(wire
 		(pts
-			(xy 44.45 97.79) (xy 44.45 93.98)
+			(xy 60.96 106.68) (xy 93.98 106.68)
 		)
 		(stroke
@@
 	(wire
 		(pts
-			(xy 60.96 106.68) (xy 93.98 106.68)
+			(xy 60.96 115.57) (xy 60.96 111.76)
 		)
 		(stroke
@@
 	(wire
 		(pts
-			(xy 125.73 73.66) (xy 107.95 73.66)
+			(xy 143.51 78.74) (xy 143.51 81.28)
 		)
 		(stroke
@@
 	(wire
 		(pts
-			(xy 60.96 115.57) (xy 60.96 111.76)
+			(xy 93.98 106.68) (xy 93.98 113.03)
 		)
 		(stroke
@@
 	(wire
 		(pts
-			(xy 143.51 78.74) (xy 143.51 81.28)
+			(xy 93.98 115.57) (xy 60.96 115.57)
 		)
 		(stroke
@@
 		)
 	)
-	(wire
-		(pts
-			(xy 125.73 71.12) (xy 125.73 73.66)
-		)
-		(stroke
-			(width 0)
-			(type default)
-		)
-	)
-	(wire
-		(pts
-			(xy 93.98 106.68) (xy 93.98 113.03)
-		)
-		(stroke
-			(width 0)
-			(type default)
-		)
-	)
-	(wire
-		(pts
-			(xy 93.98 115.57) (xy 60.96 115.57)
-		)
-		(stroke
-			(width 0)
-			(type default)
-		)
-	)
 	(global_label "ROW3"
 		(shape input)
@@
 				)
 				(justify left)
+				(hide yes)
+			)
+		)
+	)
+	(global_label "GND"
+		(shape input)
+		(at 151.13 55.88 0)
+		(fields_autoplaced yes)
+		(effects
+			(font
+				(size 1.27 1.27)
+			)
+			(justify left)
+		)
+		(property "Intersheetrefs" "${INTERSHEET_REFS}"
+			(at 157.9857 55.88 0)
+			(effects
+				(font
+					(size 1.27 1.27)
+				)
+				(justify left)
+				(hide yes)
+			)
+		)
+	)
+	(global_label "RST"
+		(shape input)
+		(at 140.97 55.88 180)
+		(fields_autoplaced yes)
+		(effects
+			(font
+				(size 1.27 1.27)
+			)
+			(justify right)
+		)
+		(property "Intersheetrefs" "${INTERSHEET_REFS}"
+			(at 134.5377 55.88 0)
+			(effects
+				(font
+					(size 1.27 1.27)
+				)
+				(justify right)
 				(hide yes)
 			)
@@
 	(symbol
 		(lib_id "Switch:SW_Push")
-		(at 120.65 71.12 0)
+		(at 146.05 55.88 0)
 		(unit 1)
 		(exclude_from_sim no)
@@
 		(fields_autoplaced yes)
 		(property "Reference" "SW99"
-			(at 120.65 63.5 0)
+			(at 146.05 48.26 0)
 			(effects
 				(font
@@
 		)
 		(property "Value" "SW_Push"
-			(at 120.65 66.04 0)
+			(at 146.05 50.8 0)
 			(effects
 				(font
@@
 		)
 		(property "Footprint" "ergogen_fp:sw_reset_side"
-			(at 120.65 66.04 0)
+			(at 146.05 50.8 0)
 			(effects
 				(font
@@
 		)
 		(property "Datasheet" "~"
-			(at 120.65 66.04 0)
+			(at 146.05 50.8 0)
 			(effects
 				(font
@@
 		)
 		(property "Description" "Push button switch, generic, two pins"
-			(at 120.65 71.12 0)
-			(effects
-				(font
+			(at 146.05 55.88 0)
+			(effects
+				(font

Commit message: inprocess
Connections:
- net COL6: now also U1.9 (P1.00)
- net GND: now also U1.14 (GND), U1.28 (GND), U1.3 (GND), U1.4 (GND)
- net ROW1: now also U1.19 (P0.02-LF); no longer U1.18 (P0.29-LF)
- net ROW2: now also U1.6 (P0.20); no longer U1.19 (P0.02-LF)
- net ROW3: now also U1.7 (P0.22); no longer U1.20 (P1.15-LF)
- net ROW4: now also U1.8 (P0.24); no longer U1.21 (P1.13-LF)
- net RST: now also U1.15 (RST)
- net EC_B: now reaches U1.10 (P0.11)
- net EC_B: now also SW98.B
- net at SW97.2 (B): no longer U1.11 (P1.04-LF)
- net EC_A: now reaches U1.12 (P1.06-LF)
- net EC_A: now also SW98.A
- net COL1: now reaches U1.22 (P1.11-LF)
- net COL2: now reaches U1.23 (P0.10-LF)
- net COL3: now reaches U1.24 (P0.09-LF)
- net at SW97.1 (C): no longer J1.2 (Pin_2)
- net at SW97.3 (A): no longer J1.1 (Pin_1)
- net EC_C: now reaches SW98.C
- net EC_C: now also U1.11 (P1.04-LF)
- new net COL0: U1.21 (P1.13-LF)
- new net COL4: U1.18 (P0.29-LF)
- new net COL5: U1.20 (P1.15-LF)
Other:
- moved on the sheet: D98, J1, SW98
