File: PCB/Keyboard/Reversible_PCB.kicad_pcb (KiCad board)
At the start: 2 copper layers, 134.8 x 110.6 mm, 71 parts, among them J1 Conn_01x02_Socket, J10 Jumper, J11 Jumper, J12 Jumper, J13 Jumper, J14 Jumper, J7 Jumper, J8 Jumper, J9 Jumper, SW1 SW_Push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

Commit message: Cleaned
Connections:
- J1 pad 1: GND -> VCC
Routing:
- net GND: track 85.2 -> 88.5 mm
- net VCC: track 39.9 -> 41.7 mm
Other:
- outline, holes or cut-outs redrawn
- board text added: "PWR"
