File: PCB/Keyboard/plate.kicad_pcb (KiCad board)
At the start: 2 copper layers, 134.8 x 110.6 mm, 28 parts, among them SW1 SW_Push, SW10 SW_Push, SW11 SW_Push, SW12 SW_Push, SW13 SW_Push, SW14 SW_Push, SW15 SW_Push, SW16 SW_Push, SW17 SW_Push, SW18 SW_Push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

Commit message: ajust plate
Other:
- board size 134.8 x 110.6 mm -> 131.1 x 110.6 mm
Changed lines of the file:
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@@
 		(fp_arc
 			(start -6.997237 -6.498884)
-			(mid -6.850789 -6.852437)
+			(mid -6.850789 -6.852436)
 			(end -6.497236 -6.998884)
 			(stroke
@@
 		(fp_arc
 			(start -6.5 7)
-			(mid -6.853554 6.853553)
+			(mid -6.853554 6.853554)
 			(end -7 6.5)
 			(stroke
@@
 	)
 	(gr_line
-		(start 183.33 115.44)
-		(end 183.33 94.149991)
-		(stroke
-			(width 0.1)
-			(type default)
-		)
-		(layer "B.SilkS")
-	)
-	(gr_line
-		(start 105.94 115.53)
-		(end 89.061663 115.53)
-		(stroke
-			(width 0.05)
-			(type default)
-		)
-		(layer "Edge.Cuts")
-	)
-	(gr_line
 		(start 174.381666 114.249982)
 		(end 174.381666 131.3)
@@
 	)
 	(gr_arc
-		(start 105.94 115.530751)
-		(mid 106.919236 116.331015)
-		(end 106.33 117.449999)
-		(stroke
-			(width 0.05)
-			(type default)
-		)
-		(layer "Edge.Cuts")
-	)
-	(gr_arc
 		(start 146.601666 35.479069)
 		(mid 146.89457 34.771982)
@@
 	)
 	(gr_arc
+		(start 108.49 115.96)
+		(mid 108.29 116.56)
+		(end 107.77 116.92)
+		(stroke
+			(width 0.05)
+			(type default)
+		)
+		(layer "Edge.Cuts")
+	)
+	(gr_arc
 		(start 222.891666 117.01)
 		(mid 222.598773 117.717107)
@@
 		(layer "Edge.Cuts")
 	)
+	(gr_line
+		(start 108.5 40.24)
+		(end 108.49 115.96)
+		(stroke
+			(width 0.05)
+			(type default)
+		)
+		(layer "Edge.Cuts")
+	)
 	(gr_arc
 		(start 174.381666 114.249982)
@@
 	(gr_line
 		(start 126.551666 39.24)
-		(end 89.061633 39.24)
-		(stroke
-			(width 0.05)
-			(type default)
-		)
-		(layer "Edge.Cuts")
-	)
-	(gr_line
-		(start 88.061633 40.24)
-		(end 88.061663 114.53)
+		(end 109.5 39.24)
 		(stroke
 			(width 0.05)
@@
 	)
 	(gr_arc
-		(start 88.061633 40.24)
-		(mid 88.354524 39.532882)
-		(end 89.061633 39.24)
-		(stroke
-			(width 0.05)
-			(type default)
-		)
-		(layer "Edge.Cuts")
-	)
-	(gr_arc
 		(start 127.55158 37.95)
 		(mid 127.844474 37.242898)
@@
 	(gr_line
 		(start 92.43 122.520001)
-		(end 106.33 117.449999)
+		(end 107.77 116.92)
 		(stroke
 			(width 0.05)
@@
 		(layer "Edge.Cuts")
 	)
-	(gr_arc
-		(start 89.061663 115.53)
-		(mid 88.354558 115.237106)
-		(end 88.061663 114.53)
-		(stroke
-			(width 0.05)
-			(type default)
-		)
-		(layer "Edge.Cuts")
-	)
 	(gr_line
 		(start 136.33 134.64)
@@
 		(layer "Edge.Cuts")
 	)
-	(gr_rect
-		(start 91.39 92.17)
-		(end 103.66 104.05)
+	(gr_line
+		(start 164.791562 34.479069)
+		(end 147.601666 34.479069)
 		(stroke
 			(width 0.05)
 			(type default)
 		)
-		(fill none)
 		(layer "Edge.Cuts")
 	)
 	(gr_line
-		(start 164.791562 34.479069)
-		(end 147.601666 34.479069)
+		(start 127.55158 37.95)
+		(end 127.55158 38.195135)
 		(stroke
 			(width 0.05)
@@
 		(layer "Edge.Cuts")
 	)
-	(gr_line
-		(start 127.55158 37.95)
-		(end 127.55158 38.195135)
+	(gr_arc
+		(start 108.5 40.24)
+		(mid 108.792893 39.532893)
+		(end 109.5 39.24)
 		(stroke
 			(width 0.05)
